File: hardware/ControlBoard/ControlBoard.kicad_pcb (KiCad board)
At the start: 4 copper layers, 95 x 95 mm, 128 parts, among them J1 Lamp 1 Out, J10 CAN, J11 USB_B_Micro, J12 Conn_01x02, J13 AVAILABLE GPIO, J14 MOTOR_CTRL1, J15 MOTOR_CTRL2, J2 ESTOP1, J3 ESTOP2, J4 Lamp 3 Out, J5 Lamp 2 Out, J6 Lamp 4 Out, J7 PWR_IN, J8 USB_B_Micro, J9 UART BACKUP, Q1 2N7002, Q2 2N7002, Q3 2N7002, Q4 2N7002, Q5 SS8050-G, Q6 SS8050-G, SW1 SW_Push, SW2 SW_Push, U1 CP2102N-A02-GQFN28, U2 Lora_Module, U3 AZ1117IH-5.0TRG1, U4 LD1086DT33TR, U5 ESP32-S3-WROOM-1U, U6 74LVC1G97W6-7, U7 SN65HVD232, U8 SN74LVC1GU04DBVR

Commit message: Motor control stuff
Parts:
- added C22: 0.1u, Capacitor_SMD:C_0805_2012Metric, F.Cu at (78.0, 102.1)
- added C23: 0.1u, Capacitor_SMD:C_0805_2012Metric, F.Cu at (73.5, 102.1)
- added C24: 0.1u, Capacitor_SMD:C_0805_2012Metric, F.Cu at (38.2, 85.8)
- added C25: 0.1u, Capacitor_SMD:C_0805_2012Metric, F.Cu at (33.7, 85.8)
- added C28: 0.1u, Capacitor_SMD:C_0805_2012Metric, F.Cu at (29.3, 88.8)
- added C29: 0.1u, Capacitor_SMD:C_0805_2012Metric, F.Cu at (66.0, 111.5)
- added R52: 10k, Resistor_SMD:R_0805_2012Metric, F.Cu at (38.2, 88.7)
- added R53: 10k, Resistor_SMD:R_0805_2012Metric, B.Cu at (75.9, 97.5)
- added R54: 680, Resistor_SMD:R_0805_2012Metric, F.Cu at (29.3, 94.8)
- added R55: 680, Resistor_SMD:R_0805_2012Metric, F.Cu at (68.8, 110.5)
- added U10: TXB0106PWR, controlLib:TXB0106PWR, F.Cu at (22.8, 88.0)
- added U9: TXB0106PWR, controlLib:TXB0106PWR, F.Cu at (75.8, 98.1)
- R33: moved to B.Cu
- moved R33 55.8 mm to (76.8, 100.4), turned to -90 degrees
- moved R32 23.4 mm to (33.7, 91.7), turned to 0 degrees
- moved R26 18.9 mm to (85.7, 99.6), turned to 180 degrees
- moved R27 17.1 mm to (85.7, 101.5), turned to 180 degrees
- moved R28 15.5 mm to (85.7, 103.5), turned to 180 degrees
- moved R38 5.46 mm to (63.3, 110.5)
- moved R34 1.48 mm to (54.7, 80.4)
- moved R35 1.38 mm to (131.3, 87.8)
Connections:
- net /ENA-_1_IO renamed /ENA-_1_IO_3V3
- net /ENA-_2_IO renamed /ENA-_2_IO_3V3
- J14 pad 1: /DIR+_1 -> /DIR+_1_5V
- J14 pad 3: /DIR+_1 -> /DIR+_1_5V
- J14 pad 5: /DIR+_1 -> /DIR+_1_5V
- J14 pad 6: /ENA-_1 -> /ENA-_1_5V
- J14 pad 7: /INP+_1 -> /INP+_1_5V
- J14 pad 9: /ALM+_1 -> /ALM+_1_5V
- R26 pad 1: /ENA-_1 -> /ENA-_1_3V3
- R27 pad 1: /ENA-_1 -> /ENA-_1_3V3
- R28 pad 1: /ENA-_1 -> /ENA-_1_3V3
- R29 pad 1: /ENA-_2 -> /ENA-_2_3V3
- R30 pad 1: /ENA-_2 -> /ENA-_2_3V3
- R31 pad 1: /ENA-_2 -> /ENA-_2_3V3
- R32 pad 1: /DIR+_1 -> Net-(R32-Pad1)
- R32 pad 2: +12V -> /ESTOP_OUT_N
- R33 pad 1: /DIR+_2 -> Net-(R33-Pad1)
- R33 pad 2: +12V -> /ESTOP_OUT_N
- R34 pad 2: /DIR+_1 -> /DIR+_1_5V
- R36 pad 1: /ALM+_1 -> /ALM+_1_5V
- R38 pad 2: /PUL-_1 -> /PUL-_1_5V
- R39 pad 2: /DIR-_1 -> /DIR-_1_5V
- R42 pad 1: /INP+_1 -> /INP+_1_5V
- U5 pad 10: /DIR-_1 -> /DIR-_1_3V3
- U5 pad 11: /PUL-_1 -> /PUL-_1_3V3
- U5 pad 30: /ALM+_2 -> /ALM+_2_3V3
- U5 pad 31: /INP+_2 -> /INP+_2_3V3
- U5 pad 33: /DIR-_2 -> /DIR-_2_3V3
- U5 pad 34: /PUL-_2 -> /PUL-_2_3V3
- U5 pad 7: /ALM+_1 -> /ALM+_1_3V3
- U5 pad 8: /INP+_1 -> /INP+_1_3V3
Routing:
- net /DIR+_1: track 41.8 -> 0.00 mm
- net /DIR+_1_5V: track 0.00 -> 40.3 mm
- net /ALM+_1: track 32.2 -> 0.00 mm
- net /INP+_1: track 30.3 -> 0.00 mm
- net /PUL-_1: track 22.7 -> 0.00 mm
- net /DIR-_1: track 20.7 -> 0.00 mm
- net /ESTOP_OUT_N: track 94.0 -> 75.1 mm, vias 3 -> 2
- net /ENA-_1_IO_3V3: track 18.4 -> 0.00 mm
- net /ENA-_1: track 11.3 -> 0.00 mm
- net /ENA-_2_3V3: track 0.00 -> 11.3 mm
- net /ENA-_2: track 11.3 -> 0.00 mm
- net /ESTOP_OUT: track 114.9 -> 103.8 mm, vias 3 -> 2
- net /INP+_1_5V: track 0.00 -> 10.5 mm
- net Net-(J14-Pad2): track 8.38 -> 0.00 mm
- net /ALM+_1_5V: track 0.00 -> 5.16 mm
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
Commit message: Control Board Routing Work
Parts:
- R26, R27, R29, R30, R32, R52: moved to B.Cu
- moved C28 98.5 mm to (127.7, 91.3), turned to 90 degrees
- moved U10 97.3 mm to (119.6, 98.8)
- moved R54 96.5 mm to (125.7, 93.2), turned to 90 degrees
- moved C25 88.4 mm to (121.7, 94.8)
- moved R32 84.2 mm to (116.7, 106.3), turned to -90 degrees
- moved R52 80.8 mm to (117.6, 103.7)
- moved C24 79.9 mm to (117.5, 94.8), turned to 180 degrees
- moved R30 14.3 mm to (112.0, 102.7), turned to -90 degrees
- moved R29 14.3 mm to (114.0, 102.7), turned to -90 degrees
- moved R31 13.8 mm to (110.5, 99.1), turned to 180 degrees
- moved TP3 12.5 mm to (83.1, 77.2)
- moved R26 4.98 mm to (81.7, 102.5), turned to -90 degrees
- moved R28 4.54 mm to (84.2, 99.2), turned to 0 degrees
- moved R39 3.76 mm to (65.0, 104.5)
- moved R40 3.70 mm to (129.7, 91.3), turned to -90 degrees
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Connections:
- net /DIR+_2 renamed /DIR+_2_5V
- J15 pad 6: /ENA-_2 -> /ENA-_2_5V
- J15 pad 7: /INP+_2 -> /INP+_2_5V
- J15 pad 9: /ALM+_2 -> /ALM+_2_5V
- R37 pad 1: /ALM+_2 -> /ALM+_2_5V
- R40 pad 2: /PUL-_2 -> /PUL-_2_5V
- R41 pad 2: /DIR-_2 -> /DIR-_2_5V
- R43 pad 1: /INP+_2 -> /INP+_2_5V
- U10 pad 10: /PUL-_2_5V_UF -> /ALM+_2_5V
- U10 pad 11: /DIR-_2_5V -> /INP+_2_5V
- U10 pad 13: /INP+_2_5V -> /DIR-_2_5V
- U10 pad 14: /ALM+_2_5V -> /PUL-_2_5V_UF
- U10 pad 3: /ALM+_2_3V3 -> /PUL-_2_3V3
- U10 pad 4: /INP+_2_3V3 -> /DIR-_2_3V3
- U10 pad 6: /DIR-_2_3V3 -> /INP+_2_3V3
- U10 pad 7: /PUL-_2_3V3 -> /ALM+_2_3V3
- U5 pad 41_10: (no net) -> GND
- U5 pad 41_11: (no net) -> GND
- U5 pad 41_12: (no net) -> GND
- U5 pad 41_13: (no net) -> GND
- U5 pad 41_14: (no net) -> GND
Routing:
- net +5V: track 0.00 -> 260.7 mm, vias 0 -> 19
- net GND: track 37.2 -> 214.6 mm, vias 0 -> 43
- net +12V: track 0.00 -> 57.8 mm, vias 0 -> 9
- net +3V3: track 13.8 -> 69.7 mm, vias 0 -> 21
- net /BOOT: track 5.39 -> 40.5 mm, vias 0 -> 2
- net /ALM+_2: track 32.9 -> 0.00 mm
- net /INP+_2: track 30.9 -> 0.00 mm
- net /CHIP_PU: track 16.2 -> 44.8 mm, vias 0 -> 2
- net /ESTOP_OUT: track 103.8 -> 80.2 mm, vias 2 -> 1
- net /PUL-_2: track 20.8 -> 0.00 mm
- net /DIR-_2: track 20.1 -> 0.00 mm
- net /ALM+_2_5V: track 0.00 -> 19.0 mm
- net /INP+_2_5V: track 0.00 -> 15.0 mm
- net /ENA-_2_IO_3V3: track 18.2 -> 3.44 mm
- net /ENA-_2_5V: track 0.00 -> 14.0 mm
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- added copper zone on B.Cu, net +12V
- added copper zone on F.Cu, net +12V
- added copper zone on B.Cu, net +3V3
- added copper zone on F.Cu, net +3V3
- added copper zone on B.Cu, net +5V
- added copper zone on F.Cu, net +5V
- added copper zone on F.Cu, net GND
- added copper zone on In2.Cu, net GND

Commit message: Routing Work
Parts:
- added G***: LOGO, controlLib:Paradigm_NameBelow_12.7mm, F.Cu at (74.7, 89.5)
- moved J11 0.63 mm to (53.0, 125.4)
- moved J8 0.60 mm to (141.9, 74.5)
Routing:
- net GND: track 214.6 -> 219.6 mm, vias 43 -> 49
- net /INP+_1_3V3: track 11.0 -> 10.3 mm
- net /VBUSB: track 6.87 -> 7.51 mm
- net /USB_DN: track 25.3 -> 25.9 mm
- net /VBUS: track 26.7 -> 27.2 mm
- net /USB_DP: track 25.9 -> 26.5 mm
- added copper zone on B.Cu, net GND
Other:
- board text added: "+12V"
- board text added: "+3.3V"
- board text added: "+5V"
- board text added: "ESTOP BUTTON"
- board text added: "ESTOP_M"
- board text added: "ESTOP_OUT"
- board text added: "ESTOP_W"
- board text added: "LAMP 1"
- board text added: "LAMP 2"
- board text added: "LAMP 3"
- board text added: "LAMP 4"
- board text added: "MOTOR CTRL 1"
- board text added: "MOTOR CTRL 2"
- board text added: "PWR"
- board text added: "Paradigm IGVC Control Board Rev 1 Dylan Matthews Luke Cronin 2023"
- board text added: "USB"
- board text added: "USB TO UART"

Commit message: More Control Board Routing Stuff
Routing:
- net GND: vias 49 -> 55
Other:
- board text added: "Paradigm IGVC Control Board Rev 1 Dylan Matthews | Luke Cronin 2023"
- board text removed: "Paradigm IGVC Control Board Rev 1 Dylan Matthews Luke Cronin 2023"
Changed lines of the file:
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@@
     (property "Sheetname" "")
     (attr exclude_from_pos_files)
-    (fp_text reference "H3" (at -2.975 -3.725) (layer "F.SilkS")
+    (fp_text reference "H3" (at -2.975 -3.725) (layer "F.SilkS") hide
       (effects (font (size 1 1) (thickness 0.15)))
     )
@@
     (property "Sheetname" "")
     (attr smd)
-    (fp_text reference "R6" (at 0 1.725) (layer "F.SilkS")
+    (fp_text reference "R6" (at -3.05 0) (layer "F.SilkS")
       (effects (font (size 1 1) (thickness 0.15)))
     )
@@
     (property "Sheetname" "")
     (attr smd)
-    (fp_text reference "R15" (at 2.2625 -1.7) (layer "F.SilkS")
+    (fp_text reference "R15" (at 2.4375 -1.7) (layer "F.SilkS")
       (effects (font (size 1 1) (thickness 0.15)))
     )
@@
     (pad "6" smd rect (at -0.95 -1.2 90) (size 0.55 0.8) (layers "F.Cu" "F.Paste" "F.Mask")
       (net 68 "Net-(R25-Pad2)") (pinfunction "IN2") (pintype "input"))
+    (model "${KIPRJMOD}/3D_lib/74LVC1G97W6-7.STEP"
+      (offset (xyz 0 0 0))
+      (scale (xyz 1 1 1))
+      (rotate (xyz -90 0 -90))
+    )
   )
   (footprint "Diode_SMD:D_SMA" (layer "F.Cu")
@@
     (property "Sheetname" "")
     (attr smd)
-    (fp_text reference "R2" (at 0 1.75) (layer "F.SilkS")
+    (fp_text reference "R2" (at -3.075 0) (layer "F.SilkS")
       (effects (font (size 1 1) (thickness 0.15)))
     )
@@
     (property "Sheetname" "")
     (attr exclude_from_pos_files)
-    (fp_text reference "H1" (at 0 -4.2) (layer "F.SilkS")
+    (fp_text reference "H1" (at 0 -4.2) (layer "F.SilkS") hide
       (effects (font (size 1 1) (thickness 0.15)))
     )
@@
     (pad "4" smd rect (at -3.1 0) (size 2.2 3.5) (layers "F.Cu" "F.Paste" "F.Mask")
       (net 6 "+5V") (pinfunction "VOUT") (pintype "input"))
+    (model "${KIPRJMOD}/3D_lib/SOT223-5_DIO.step"
+      (offset (xyz 0 0 0))
+      (scale (xyz 1 1 1))
+      (rotate (xyz 0 0 -90))
+    )
   )
   (footprint "Resistor_SMD:R_0805_2012Metric" (layer "F.Cu")
@@
     (pad "3" smd rect (at 9.3 -2.286 90) (size 2.8 1.5) (layers "F.Cu" "F.Paste" "F.Mask")
       (net 5 "+12V") (pinfunction "IN") (pintype "power_in"))
+    (model "${KIPRJMOD}/3D_lib/LD1086DT33TR.STEP"
+      (offset (xyz 5.25 0 0))
+      (scale (xyz 1 1 1))
+      (rotate (xyz -90 0 180))
+    )
   )
   (footprint "Connector_Molex:Molex_Micro-Fit_3.0_43650-0200_1x02_P3.00mm_Horizontal" (layer "F.Cu")
@@
     (pad "41_9" thru_hole circle (at -0.1 0.01) (size 0.45 0.45) (drill 0.3) (layers *.Cu)
       (net 2 "GND") (pinfunction "GND") (pintype "power_in"))
+    (model "${KIPRJMOD}/3D_lib/ESP32-S3-WROOM-1U--3DModel-STEP-56544.STEP"
+      (offset (xyz 0 0 0))
+      (scale (xyz 1 1 1))
+      (rotate (xyz -90 0 0))
+    )
   )
   (footprint "Button_Switch_SMD:SW_SPST_B3U-1100P-B" (layer "F.Cu")
@@
     (property "Sheetname" "")
     (attr smd)
-    (fp_text reference "SW1" (at -2.55 1.58 90) (layer "F.SilkS")
+    (fp_text reference "SW1" (at -1.625 2.48 180) (layer "F.SilkS")
       (effects (font (size 1 1) (thickness 0.15)))
     )
@@
     (property "Sheetname" "")
     (attr smd)
-    (fp_text reference "R41" (at 0 -1.725) (layer "F.SilkS")
+    (fp_text reference "R41" (at -0.725 -1.75) (layer "F.SilkS")
       (effects (font (size 1 1) (thickness 0.15)))
     )
@@
     (property "Sheetname" "")
     (attr smd)
-    (fp_text reference "R1" (at 0.025 1.925) (layer "F.SilkS")
+    (fp_text reference "R1" (at -3.15 0) (layer "F.SilkS")
       (effects (font (size 1 1) (thickness 0.15)))
     )
@@
     (property "Sheetname" "")
     (attr exclude_from_pos_files)
-    (fp_text reference "TP6" (at 2.9 -1.225) (layer "F.SilkS")
+    (fp_text reference "TP6" (at 2.225 -0.6 -270) (layer "F.SilkS")
       (effects (font (size 1 1) (thickness 0.15)))
     )
@@
     (property "Sheetname" "")
     (attr exclude_from_pos_files)
-    (fp_text reference "TP3" (at 2.65 -1) (layer "F.SilkS")
+    (fp_text reference "TP3" (at 2.425 0) (layer "F.SilkS")
       (effects (font (size 1 1) (thickness 0.15)))
     )
@@
     (property "Sheetname" "")
     (attr smd)
-    (fp_text reference "J11" (at 5.35 0.025) (layer "F.SilkS")
+    (fp_text reference "J11" (at 5.2 -1.41) (layer "F.SilkS")
       (effects (font (size 1 1) (thickness 0.15)))
     )
@@
   (gr_line (start 50 145) (end 145 145) (layer "Edge.Cuts") (width 0.1))
   (gr_line (start 145 50) (end 50 50) (layer "Edge.Cuts") (width 0.1))
-  (gr_text "ESTOP_W" (at 88.625 130.8) (layer "F.SilkS")
+  (gr_text "ESTOP_W" (at 87.75 131.75 -270) (layer "F.SilkS")
     (effects (font (size 1 1) (thickness 0.15)))
   )
@@
     (effects (font (size 1 1) (thickness 0.15)))
   )
-  (gr_text "USB" (at 57.375 128.05 -90) (layer "F.SilkS")
+  (gr_text "USB" (at 51.575 131.75 -90) (layer "F.SilkS")
     (effects (font (size 1 1) (thickness 0.15)))
   )
@@
     (effects (font (size 1 1) (thickness 0.15)))
   )
-  (gr_text "Paradigm IGVC\nControl Board Rev 1\nDylan Matthews\nLuke Cronin\n2023" (at 100.45 76.875) (layer "F.SilkS")
+  (gr_text "Paradigm IGVC\nControl Board Rev 1\nDylan Matthews | Luke Cronin\n2023" (at 99.45 74.2) (layer "F.SilkS")
     (effects (font (size 1 1) (thickness 0.15)))
   )
-  (gr_text "+3.3V" (at 86.25 77.825) (layer "F.SilkS")
+  (gr_text "+3.3V" (at 85.3 78.825) (layer "F.SilkS")
     (effects (font (size 1 1) (thickness 0.15)))
   )
@@
   (via (at 60.15 74.55) (size 0.8) (drill 0.4) (layers "F.Cu" "B.Cu") (net 2))
   (via (at 122.6 93.175) (size 0.8) (drill 0.4) (layers "F.Cu" "B.Cu") (net 2))
+  (via (at 63.075 106.775) (size 0.8) (drill 0.4) (layers "F.Cu" "B.Cu") (net 2))
   (via (at 143 63.925) (size 0.8) (drill 0.4) (layers "F.Cu" "B.Cu") (net 2))
   (via (at 74.45 96.1) (size 0.8) (drill 0.4) (layers "F.Cu" "B.Cu") (net 2))
@@
   (via (at 110.625 107.825) (size 0.8) (drill 0.4) (layers "F.Cu" "B.Cu") (net 2))
   (via (at 115.325 77.7) (size 0.8) (drill 0.4) (layers "F.Cu" "B.Cu") (free) (net 2))
+  (via (at 64.825 97.675) (size 0.8) (drill 0.4) (layers "F.Cu" "B.Cu") (net 2))
   (via (at 85.55 106.95) (size 0.8) (drill 0.4) (layers "F.Cu" "B.Cu") (free) (net 2))
   (via (at 127.45 87.925) (size 0.8) (drill 0.4) (layers "F.Cu" "B.Cu") (net 2))
@@
   (via (at 82.325 124.1) (size 0.8) (drill 0.4) (layers "F.Cu" "B.Cu") (net 2))
   (via (at 72.875 96.075) (size 0.8) (drill 0.4) (layers "F.Cu" "B.Cu") (net 2))
+  (via (at 62.55 101.375) (size 0.8) (drill 0.4) (layers "F.Cu" "B.Cu") (net 2))
   (via (at 51.725 60.875) (size 0.8) (drill 0.4) (layers "F.Cu" "B.Cu") (net 2))
   (via (at 93.125 81.125) (size 0.8) (drill 0.4) (layers "F.Cu" "B.Cu") (net 2))
   (via (at 133.5 80.575) (size 0.8) (drill 0.4) (layers "F.Cu" "B.Cu") (net 2))
+  (via (at 127.65 97.95) (size 0.8) (drill 0.4) (layers "F.Cu" "B.Cu") (net 2))
   (via (at 116.575 93.15) (size 0.8) (drill 0.4) (layers "F.Cu" "B.Cu") (net 2))
+  (via (at 126.675 102.325) (size 0.8) (drill 0.4) (layers "F.Cu" "B.Cu") (net 2))
   (via (at 66.05 113.8) (size 0.8) (drill 0.4) (layers "F.Cu" "B.Cu") (net 2))
+  (via (at 129.225 93.775) (size 0.8) (drill 0.4) (layers "F.Cu" "B.Cu") (net 2))
   (via (at 89.85 80.525) (size 0.8) (drill 0.4) (layers "F.Cu" "B.Cu") (net 2))
   (via (at 69.575 131.95) (size 0.8) (drill 0.4) (layers "F.Cu" "B.Cu") (net 2))

Commit message: Most control board schematic fixes done
Parts:
- removed G***: LOGO, controlLib:Paradigm_NameBelow_12.7mm
- added C30: 10n, Capacitor_SMD:C_0805_2012Metric, F.Cu at (121.7, 22.6)
- added C31: 1u, Capacitor_SMD:C_0805_2012Metric, F.Cu at (121.0, 28.6)
- added C32: 0.1u, Capacitor_SMD:C_0805_2012Metric, F.Cu at (113.3, 35.2)
- added C33: 0.1u, Capacitor_SMD:C_0805_2012Metric, F.Cu at (104.5, 36.5)
- added C34: 1u, Capacitor_SMD:C_0805_2012Metric, F.Cu at (126.0, 18.1)
- added C35: 0.1u, Capacitor_SMD:C_0805_2012Metric, F.Cu at (100.2, 41.0)
- added C36: 0.1u, Capacitor_SMD:C_0805_2012Metric, F.Cu at (125.4, 25.6)
- added C37: 1u, Capacitor_SMD:C_0805_2012Metric, F.Cu at (121.0, 25.6)
- added C38: 0.1u, Capacitor_SMD:C_0805_2012Metric, F.Cu at (126.1, 21.1)
- added C39: 0.1u, Capacitor_SMD:C_0805_2012Metric, F.Cu at (104.6, 39.5)
- added C40: 1u, Capacitor_SMD:C_0805_2012Metric, F.Cu at (108.9, 36.5)
- added R56: 2k, Resistor_SMD:R_0805_2012Metric, F.Cu at (139.2, 18.0)
- added R57: 4.7k, Resistor_SMD:R_0805_2012Metric, F.Cu at (117.9, 41.0)
- added R58: 4.7k, Resistor_SMD:R_0805_2012Metric, F.Cu at (113.5, 41.1)
- added R59: 4.7k, Resistor_SMD:R_0805_2012Metric, F.Cu at (125.4, 28.6)
- added R60: 0, Resistor_SMD:R_0805_2012Metric, F.Cu at (129.8, 24.1)
- added R61: 10k, Resistor_SMD:R_0805_2012Metric, F.Cu at (130.5, 21.0)
- added R62: 0, Resistor_SMD:R_0805_2012Metric, F.Cu at (113.5, 38.1)
- added R63: 0, Resistor_SMD:R_0805_2012Metric, F.Cu at (117.9, 38.0)
- added R64: 0, Resistor_SMD:R_0805_2012Metric, F.Cu at (118.3, 32.1)
- added R65: 10k, Resistor_SMD:R_0805_2012Metric, F.Cu at (127.1, 31.5)
- added R66: 0, Resistor_SMD:R_0805_2012Metric, F.Cu at (129.8, 27.0)
- added R67: 0, Resistor_SMD:R_0805_2012Metric, F.Cu at (134.9, 21.0)
- added U11: 74LVC1G17W5-7, controlLib:74LVC1G17W5-7, F.Cu at (104.1, 24.9)
- added U12: TXU0104QPWRQ1, controlLib:TXU0104QPWRQ1, F.Cu at (114.5, 27.7)
- C15, C16: value 0.1uF -> 0.1u
- C17: value 10nF -> 0.1u
- C5: value 10u -> 22u
- J11, J8: footprint Connector_USB:USB_Micro-B_Molex-105017-0001 -> Connector_USB:USB_Micro-B_Amphenol_10118194_Horizontal
- Q1, Q2, Q3, Q4: value 2N7002 -> DMN62D0U-13; footprint Package_TO_SOT_SMD:SOT-23 -> controlLib:DMN62D0U-13
- R32, R33: value 0 -> 220; moved to F.Cu
- R36, R37, R42, R43: value 4.7k -> 1k
- R49: value 4.7k -> 220
- R52: value 10k -> 220; moved to F.Cu
- R53: value 10k -> 1k; moved to F.Cu
- U10: value TXB0106PWR -> 74LVC1G17W5-7; footprint controlLib:TXB0106PWR -> controlLib:74LVC1G17W5-7
- U3: value AZ1117IH-5.0TRG1 -> L4941BV; footprint controlLib:AZ1117IH-5.0TRG1 -> Package_TO_SOT_THT:TO-220-3_Vertical
- U4: value LD1086DT33TR -> LD1086V33-DG; footprint controlLib:LD1086DT33TR -> Package_TO_SOT_THT:TO-220-3_Vertical
- U5: value ESP32-S3-WROOM-1U -> ESP32-S3-WROOM-1U-N16
- U9: value TXB0106PWR -> TXU0104QPWRQ1; footprint controlLib:TXB0106PWR -> controlLib:TXU0104QPWRQ1
- moved J11 122.3 mm to (114.5, 19.7), turned to 0 degrees
- moved R53 81.9 mm to (122.7, 31.6), turned to 0 degrees
- moved C25 77.2 mm to (130.4, 18.1)
- moved U10 76.5 mm to (99.8, 24.9)
- moved U9 72.6 mm to (102.9, 32.1), turned to 0 degrees
- moved R49 66.9 mm to (105.8, 68.8)
- moved C24 62.8 mm to (113.9, 32.1), turned to 0 degrees
- moved R33 52.2 mm to (115.7, 66.9)
- moved U4 48.5 mm to (83.5, 31.4), turned to 0 degrees
- moved R32 44.0 mm to (93.8, 68.8)
- moved R52 38.1 mm to (127.5, 66.9), turned to -90 degrees
- moved C22 36.0 mm to (68.2, 68.7)
- moved C23 29.6 mm to (63.1, 75.6), turned to 0 degrees
- moved U3 3.31 mm to (60.3, 68.0), turned to 180 degrees
- moved R6 1.45 mm to (107.8, 68.8), turned to 90 degrees
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Connections:
- C22 pad 1: +3V3 -> GND
- C22 pad 2: GND -> +12V
- C23 pad 1: +5V -> GND
- C23 pad 2: GND -> +5V
- C24 pad 1: +3V3 -> GND
- C24 pad 2: GND -> +12V
- C25 pad 1: +5V -> +3V3
- C28 pad 1: /PUL-_2_5V -> Net-(C28-Pad1)
- C29 pad 1: /PUL-_1_5V -> Net-(C29-Pad1)
- J14 pad 7: /INP+_1_5V -> /INP+_1_3V3
- J14 pad 9: /ALM+_1_5V -> /ALM+_1_3V3
- J15 pad 7: /INP+_2_5V -> /INP+_2_3V3
- J15 pad 9: /ALM+_2_5V -> /ALM+_2_3V3
- Q1 pad 1: /LAMP1_ON -> Net-(Q1-Pad1)
- Q2 pad 1: /LAMP3_ON -> Net-(Q2-Pad1)
- Q3 pad 1: /LAMP2_ON -> Net-(Q3-Pad1)
- Q4 pad 1: /LAMP4_ON -> Net-(Q4-Pad1)
- R32 pad 1: Net-(R32-Pad1) -> Net-(Q1-Pad1)
- R32 pad 2: /ESTOP_OUT_N -> /LAMP1_ON
- R33 pad 1: Net-(R33-Pad1) -> Net-(Q2-Pad1)
- R33 pad 2: /ESTOP_OUT_N -> /LAMP3_ON
- R36 pad 1: /ALM+_1_5V -> /ALM+_1_3V3
- R36 pad 2: +5V -> +3V3
- R37 pad 1: /ALM+_2_5V -> /ALM+_2_3V3
- R37 pad 2: +5V -> +3V3
- R42 pad 1: /INP+_1_5V -> /INP+_1_3V3
- R42 pad 2: +5V -> +3V3
- R43 pad 1: /INP+_2_5V -> /INP+_2_3V3
- R43 pad 2: +5V -> +3V3
- R49 pad 1: /ESTOP_W -> Net-(Q3-Pad1)
- R49 pad 2: GND -> /LAMP2_ON
- R52 pad 1: Net-(R32-Pad1) -> Net-(Q4-Pad1)
- R52 pad 2: GND -> /LAMP4_ON
- R53 pad 1: Net-(R33-Pad1) -> /ESTOP_W
- R53 pad 2: GND -> Net-(U2-Pad34)
- R54 pad 2: /PUL-_2_5V -> Net-(C28-Pad1)
- R55 pad 2: /PUL-_1_5V -> Net-(C29-Pad1)
- U10 pad 1: GND -> unconnected-(U10-Pad1)
- U10 pad 2: +3V3 -> Net-(C29-Pad1)
- U10 pad 3: /PUL-_2_3V3 -> GND
- U10 pad 4: /DIR-_2_3V3 -> /PUL-_1_5V
- U10 pad 5: /ENA-_2_3V3 -> +5V
- U2 pad 34: /ESTOP_W -> Net-(U2-Pad34)
- U3 pad 1: GND -> +12V
- U3 pad 2: +5V -> GND
- U3 pad 3: +12V -> +5V
- U5 pad 15: /LED1 -> unconnected-(U5-Pad15)
- U5 pad 16: /ESTOP_OUT -> Net-(U5-Pad16)
- U5 pad 17: /GPIO9 -> /ESTOP_OUT
- U5 pad 18: /GPIO10 -> /LED1
- U5 pad 24: /GPIO47 -> /CAN_RX
- U5 pad 25: /CAN_RX -> /CAN_TX
- U5 pad 26: /CAN_TX -> Net-(U5-Pad26)
- U9 pad 1: GND -> +3V3
- U9 pad 10: /ALM+_1_5V -> /ENA-_1_5V
- U9 pad 11: /INP+_1_5V -> /DIR-_1_5V
- U9 pad 12: /ENA-_1_5V -> /PUL-_1_5V_UF
- U9 pad 13: /DIR-_1_5V -> Net-(R62-Pad1)
- U9 pad 14: /PUL-_1_5V_UF -> +5V
- U9 pad 2: +3V3 -> Net-(R60-Pad2)
- U9 pad 6: /INP+_1_3V3 -> unconnected-(U9-Pad6)
- U9 pad 7: /ALM+_1_3V3 -> GND
- U9 pad 8: Net-(R33-Pad1) -> Net-(R61-Pad1)
- U9 pad 9: GND -> unconnected-(U9-Pad9)
Routing:
- net GND: track 219.6 -> 191.5 mm, vias 55 -> 51
- net +3V3: track 69.6 -> 49.9 mm, vias 21 -> 11
- net /ALM+_2_3V3: track 11.0 -> 30.0 mm
- net /ALM+_2_5V: track 19.0 -> 0.00 mm
- net /ALM+_1_5V: track 17.3 -> 0.00 mm
- net /ALM+_1_3V3: track 10.5 -> 27.8 mm
- net /INP+_2_3V3: track 10.7 -> 25.7 mm
- net /INP+_2_5V: track 15.0 -> 0.00 mm
- net /INP+_1_3V3: track 10.3 -> 24.9 mm
- net /INP+_1_5V: track 14.6 -> 0.00 mm
- net (no net): track 0.00 -> 11.1 mm, vias 0 -> 2
- net +5V: track 260.7 -> 251.2 mm, vias 19 -> 9
- net Net-(R33-Pad1): track 6.71 -> 0.00 mm, vias 1 -> 0
- net +12V: track 57.8 -> 52.5 mm, vias 9 -> 0
- net /CAN_TX: track 2.65 -> 7.50 mm
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- removed copper zone on B.Cu, net +12V
- removed copper zone on F.Cu, net +12V
- removed copper zone on F.Cu, net +3V3
- removed copper zone on B.Cu, net +5V
- removed copper zone on F.Cu, net +5V
Other:
- board text added: "heat sink"
