File: hardware/EStopTX/EStopTX/EStopTX.kicad_pcb (KiCad board)
At the start: 2 copper layers, 0 parts

Commit message: continue board
Parts:
- added C1: 100n, Capacitor_SMD:C_0805_2012Metric, F.Cu at (165.1, 83.8)
- added C1: 100n, Capacitor_THT:CP_Radial_D4.0mm_P2.00mm, F.Cu at (165.1, 58.4)
- added C2: 100n, Capacitor_THT:CP_Radial_D4.0mm_P2.00mm, F.Cu at (144.8, 83.8)
- added G***: LOGO, controlLib:Paradigm_NameBelow_12.7mm, F.Cu at (223.5, 101.6)
- added J1: USB_B, Connector_USB:USB_B_OST_USB-B1HSxx_Horizontal, F.Cu at (142.2, 63.5)
- added J2: Conn, Connector_Molex:Molex_Micro-Fit_3.0_43650-0200_1x02_P3.00mm_Horizontal, F.Cu at (179.3, 94.7)
- added R1: 4.7k, Resistor_THT:R_Axial_DIN0207_L6.3mm_D2.5mm_P10.16mm_Horizontal, F.Cu at (160.0, 96.5)
- added U2: Lora_Module, controlLib:Lora_Module, F.Cu at (224.2, 57.1)
Other:
- board text added: "Paradigm IGVC E-Stop TX Rev 1 Noel Rowsell 2023"
