File: hardware/EStopTX/EStopTX/EStopTX.kicad_pcb (KiCad board)
At the start: 2 copper layers, 8 parts, among them J1 USB_B, J2 Conn, U2 Lora_Module

Commit message: Things
Parts:
- removed the C1 at (165.1, 83.8)
- removed the G*** at (223.5, 101.6)
- removed U2: Lora_Module, controlLib:Lora_Module
- added G***: LOGO, EStopFootprints:Paradigm_NameBelow_25.4mm, F.Cu at (223.4, 71.2)
- added U1: Lora_Module, EStopFootprints:Lora_Module, F.Cu at (164.1, 60.6)
- C1, C2: footprint Capacitor_THT:CP_Radial_D4.0mm_P2.00mm -> Capacitor_THT:C_Disc_D3.8mm_W2.6mm_P2.50mm
- moved C2 49.8 mm to (191.6, 66.7)
- moved J2 35.9 mm to (143.6, 99.2)
- moved R1 13.6 mm to (148.3, 89.5)
- moved J1 9.78 mm to (151.3, 67.2), turned to 180 degrees
- moved C1 8.43 mm to (158.4, 63.6), turned to -90 degrees
Connections:
- C1 pad 1: +5V -> GND
- C1 pad 2: GND -> +5V

Commit message: maybe done?
Parts:
- added H1: MountingHole, MountingHole:MountingHole_3.2mm_M3_Pad_Via, F.Cu at (105.0, 55.0)
- added H2: MountingHole, MountingHole:MountingHole_3.2mm_M3_Pad_Via, F.Cu at (170.0, 55.0)
- added H3: MountingHole, MountingHole:MountingHole_3.2mm_M3_Pad_Via, F.Cu at (105.0, 109.0)
- added H4: MountingHole, MountingHole:MountingHole_3.2mm_M3_Pad_Via, F.Cu at (170.0, 109.0)
- moved G*** 108.0 mm to (116.8, 88.9)
- moved J2 37.1 mm to (169.1, 72.2)
- moved U1 34.7 mm to (129.5, 58.4)
- moved C2 34.6 mm to (157.5, 61.0), turned to 90 degrees
- moved C1 34.4 mm to (124.5, 58.5)
- moved J1 33.0 mm to (118.3, 69.8)
- moved R1 11.5 mm to (157.5, 96.5), turned to 90 degrees
Routing:
- net +5V: track 0.00 -> 37.9 mm
- net Net-(J2-Pad2): track 0.00 -> 33.0 mm
- added copper zone on B.Cu, net GND
- added copper zone on F.Cu, net GND
Other:
- board outline added: 75 x 64.3 mm

Commit message: updates
Parts:
- ESTOP BUTTON: renamed from J2
- moved ESTOP BUTTON 12.6 mm to (164.9, 84.1), turned to -90 degrees
- moved H3 5.00 mm to (105.0, 104.0)
- moved H4 5.00 mm to (170.0, 104.0)
- moved LORA 1.91 mm to (129.5, 56.5)
- moved PWR 1.85 mm to (116.6, 70.3)
- moved G*** 1.55 mm to (118.4, 88.6)
- renumbered U1 to LORA, J1 to PWR
Routing:
- net Net-(J2-Pad2): track 33.0 -> 18.1 mm
- net +5V: track 37.9 -> 50.6 mm
Other:
- board size 75 x 64.3 mm -> 75 x 59 mm
Changed lines of the file:
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@@
   (net 35 "unconnected-(U1-Pad36)")
   (footprint "EStopFootprints:Paradigm_NameBelow_25.4mm" (layer "F.Cu")
-    (at 116.84 88.9)
+    (at 118.364 88.646)
     (attr through_hole)
     (fp_text reference "G***" (at 0 0) (layer "F.SilkS") hide
@@
     (property "Sheetname" "")
     (attr exclude_from_pos_files)
-    (fp_text reference "H2" (at 0 -4.2) (layer "F.SilkS")
+    (fp_text reference "H2" (at 0 -4.2) (layer "F.SilkS") hide
       (effects (font (size 1 1) (thickness 0.15)))
     )
@@
   )
   (footprint "MountingHole:MountingHole_3.2mm_M3_Pad_Via" (layer "F.Cu")
-    (at 105 109)
+    (at 105 104)
     (descr "Mounting Hole 3.2mm, M3")
     (tags "mounting hole 3.2mm m3")
     (property "Sheetfile" "EStopTX.kicad_sch")
     (property "Sheetname" "")
-    (fp_text reference "H3" (at 0 -4.2) (layer "F.SilkS")
+    (fp_text reference "H3" (at 0 -4.2) (layer "F.SilkS") hide
       (effects (font (size 1 1) (thickness 0.15)))
     )
@@
   )
   (footprint "Connector_USB:USB_B_OST_USB-B1HSxx_Horizontal" (layer "F.Cu")
-    (at 118.3375 69.83 180)
+    (at 116.5595 70.338 180)
     (descr "USB B receptacle, Horizontal, through-hole, http://www.on-shore.com/wp-content/uploads/2015/09/usb-b1hsxx.pdf")
     (tags "USB-B receptacle horizontal through-hole")
@@
     (property "Sheetname" "")
     (attr through_hole)
-    (fp_text reference "J1" (at 6.76 -7.77) (layer "F.SilkS")
+    (fp_text reference "PWR" (at 6.76 -7.77) (layer "F.SilkS")
       (effects (font (size 1 1) (thickness 0.15)))
     )
@@
   )
   (footprint "MountingHole:MountingHole_3.2mm_M3_Pad_Via" (layer "F.Cu")
-    (at 170 109)
+    (at 170 104)
     (descr "Mounting Hole 3.2mm, M3")
     (tags "mounting hole 3.2mm m3")
@@
     (property "Sheetname" "")
     (attr exclude_from_pos_files)
-    (fp_text reference "H4" (at 0 -4.2) (layer "F.SilkS")
+    (fp_text reference "H4" (at 0 -4.2) (layer "F.SilkS") hide
       (effects (font (size 1 1) (thickness 0.15)))
     )
@@
   )
   (footprint "EStopFootprints:Lora_Module" (layer "F.Cu")
-    (at 129.54 58.42)
+    (at 129.54 56.51)
     (property "Sheetfile" "EStopTX.kicad_sch")
     (property "Sheetname" "")
     (attr through_hole)
-    (fp_text reference "U1" (at 11.8 -5.3 unlocked) (layer "F.SilkS")
+    (fp_text reference "LORA" (at 11.8 -5.3 unlocked) (layer "F.SilkS")
       (effects (font (size 1 1) (thickness 0.15)))
     )
@@
   )
   (footprint "Connector_Molex:Molex_Micro-Fit_3.0_43650-0200_1x02_P3.00mm_Horizontal" (layer "F.Cu")
-    (at 169.14 72.23 180)
+    (at 164.94 84.098 -90)
     (descr "Molex Micro-Fit 3.0 Connector System, 43650-0200 (compatible alternatives: 43650-0201, 43650-0202), 2 Pins per row (https://www.molex.com/pdm_docs/sd/436500300_sd.pdf), generated with kicad-footprint-generator")
     (tags "connector Molex Micro-Fit_3.0 top entry")
@@
     (property "Sheetname" "")
     (attr through_hole)
-    (fp_text reference "J2" (at 1.5 -10.12) (layer "F.SilkS")
+    (fp_text reference "ESTOP BUTTON" (at 8.358 -4.224) (layer "F.SilkS")
       (effects (font (size 1 1) (thickness 0.15)))
     )
-    (fp_text value "Conn" (at 1.5 3.22) (layer "F.Fab")
+    (fp_text value "Conn" (at 1.5 3.22 -270) (layer "F.Fab")
       (effects (font (size 1 1) (thickness 0.15)))
     )
-    (fp_text user "${REFERENCE}" (at 1.5 -8.22) (layer "F.Fab")
+    (fp_text user "${REFERENCE}" (at 1.5 -8.22 -270) (layer "F.Fab")
       (effects (font (size 1 1) (thickness 0.15)))
     )
@@
     (fp_line (start -3.325 0.98) (end -3.325 -7.92) (layer "F.Fab") (width 0.1))
     (fp_line (start 0 0) (end 0.75 0.98) (layer "F.Fab") (width 0.1))
-    (pad "" np_thru_hole circle (at 1.5 -4.32 180) (size 3 3) (drill 3) (layers *.Cu *.Mask))
-    (pad "1" thru_hole roundrect (at 0 0 180) (size 1.5 2.02) (drill 1.02) (layers *.Cu *.Mask) (roundrect_rratio 0.166667)
+    (pad "" np_thru_hole circle (at 1.5 -4.32 270) (size 3 3) (drill 3) (layers *.Cu *.Mask))
+    (pad "1" thru_hole roundrect (at 0 0 270) (size 1.5 2.02) (drill 1.02) (layers *.Cu *.Mask) (roundrect_rratio 0.166667)
       (net 1 "+5V") (pinfunction "Pin_1") (pintype "passive"))
-    (pad "2" thru_hole oval (at 3 0 180) (size 1.5 2.02) (drill 1.02) (layers *.Cu *.Mask)
+    (pad "2" thru_hole oval (at 3 0 270) (size 1.5 2.02) (drill 1.02) (layers *.Cu *.Mask)
       (net 5 "Net-(J2-Pad2)") (pinfunction "Pin_2") (pintype "passive"))
     (model "${KIPRJMOD}/Parts/3d models/436500200--3DModel-STEP-390490.STEP"
@@
     (property "Sheetname" "")
     (attr exclude_from_pos_files)
-    (fp_text reference "H1" (at 0 -4.2) (layer "F.SilkS")
+    (fp_text reference "H1" (at 0 -4.2) (layer "F.SilkS") hide
       (effects (font (size 1 1) (thickness 0.15)))
     )
@@
     )
   )
-  (gr_line (start 175 50) (end 175 114.3) (layer "Edge.Cuts") (width 0.15))
-  (gr_line (start 100 114.3) (end 175 114.3) (layer "Edge.Cuts") (width 0.15))
-  (gr_line (start 100 50) (end 100 114.3) (layer "Edge.Cuts") (width 0.15))
+  (gr_line (start 175 50) (end 175 109) (layer "Edge.Cuts") (width 0.15))
+  (gr_line (start 100 109) (end 175 109) (layer "Edge.Cuts") (width 0.15))
+  (gr_line (start 100 50) (end 100 109) (layer "Edge.Cuts") (width 0.15))
   (gr_line (start 175 50) (end 100 50) (layer "Edge.Cuts") (width 0.15))
-  (gr_text "Paradigm IGVC\nE-Stop TX Rev 1\nNoel Rowsell\n2023\n" (at 116.84 104.14) (layer "F.SilkS")
+  (gr_text "Paradigm IGVC\nE-Stop TX Rev 1\nNoel Rowsell\n2023\n" (at 117.856 102.616) (layer "F.SilkS")
     (effects (font (size 1 1) (thickness 0.15)))
   )
-  (segment (start 168.75 72.23) (end 169.14 72.23) (width 0.5) (layer "F.Cu") (net 1))
-  (segment (start 152.4 60.96) (end 157.48 60.96) (width 0.5) (layer "F.Cu") (net 1))
-  (segment (start 157.48 60.96) (end 168.75 72.23) (width 0.5) (layer "F.Cu") (net 1))
-  (segment (start 124.46 63.7075) (end 124.46 60.96) (width 0.5) (layer "F.Cu") (net 1))
-  (segment (start 129.54 60.96) (end 124.46 60.96) (width 0.5) (layer "F.Cu") (net 1))
-  (segment (start 118.3375 69.83) (end 124.46 63.7075) (width 0.5) (layer "F.Cu") (net 1))
-  (segment (start 157.48 96.52) (end 158.605 95.395) (width 0.25) (layer "F.Cu") (net 5))
-  (segment (start 158.605 95.395) (end 158.605 79.765) (width 0.25) (layer "F.Cu") (net 5))
-  (segment (start 158.605 79.765) (end 166.14 72.23) (width 0.25) (layer "F.Cu") (net 5))
-  (segment (start 152.4 96.52) (end 157.48 96.52) (width 0.25) (layer "F.Cu") (net 5))
+  (segment (start 124.46 60.96) (end 124.46 62.4375) (width 0.5) (layer "F.Cu") (net 1))
+  (segment (start 124.46 62.4375) (end 116.5595 70.338) (width 0.5) (layer "F.Cu") (net 1))
+  (segment (start 152.4 59.05) (end 154.31 60.96) (width 0.5) (layer "F.Cu") (net 1))
+  (segment (start 129.54 59.05) (end 127.63 60.96) (width 0.5) (layer "F.Cu") (net 1))
+  (segment (start 127.63 60.96) (end 124.46 60.96) (width 0.5) (layer "F.Cu") (net 1))
+  (segment (start 157.48 76.638) (end 157.48 60.96) (width 0.5) (layer "F.Cu") (net 1))
+  (segment (start 164.94 84.098) (end 157.48 76.638) (width 0.5) (layer "F.Cu") (net 1))
+  (segment (start 154.31 60.96) (end 157.48 60.96) (width 0.5) (layer "F.Cu") (net 1))
+  (segment (start 154 94.61) (end 157.48 96.52) (width 0.25) (layer "F.Cu") (net 5))
+  (segment (start 152.4 94.61) (end 154 94.61) (width 0.25) (layer "F.Cu") (net 5))
+  (segment (start 164.94 87.098) (end 164.94 89.06) (width 0.25) (layer "F.Cu") (net 5))
+  (segment (start 164.94 89.06) (end 157.48 96.52) (width 0.25) (layer "F.Cu") (net 5))
   (zone (net 2) (net_name "GND") (layers F&B.Cu) (hatch edge 0.508)
     (connect_pads (clearance 0.508))
@@
         (xy 98.552 48.768)
         (xy 176.276 48.768)
-        (xy 176.276 115.824)
-        (xy 98.552 115.824)
+        (xy 176.276 110.236)
+        (xy 98.552 110.236)
       )
     )

Commit message: adjustments
Parts:
- moved H2 57.7 mm to (112.9, 46.9), turned to 90 degrees
- moved H4 57.7 mm to (161.9, 46.9), turned to 90 degrees
- moved H1 57.5 mm to (112.9, 111.9), turned to 90 degrees
- moved H3 57.5 mm to (161.9, 111.9), turned to 90 degrees
- moved ESTOP BUTTON 39.5 mm to (142.0, 52.0), turned to 0 degrees
- moved C2 38.6 mm to (118.9, 59.4), turned to 180 degrees
- moved R1 37.2 mm to (154.4, 59.4), turned to 180 degrees
- moved C1 34.9 mm to (116.4, 92.5), turned to 0 degrees
- moved LORA 34.4 mm to (114.4, 87.4), turned to 90 degrees
- moved G*** 32.5 mm to (147.8, 102.4)
- moved PWR 32.2 mm to (128.2, 100.4), turned to -90 degrees
Other:
- board size 75 x 59 mm -> 59 x 75 mm

Commit message: changes
Parts:
- removed G***: LOGO, EStopFootprints:Paradigm_NameBelow_25.4mm
- added Switch1: L102021ML04Q, EStopFootprints:SW_L102021ML04Q, F.Cu at (149.6, 106.4)
- J2: renamed from ESTOP BUTTON
- moved J2 13.6 mm to (155.5, 50.2)
- moved R1 8.75 mm to (162.3, 63.2)
- moved J1 8.54 mm to (120.4, 103.7)
- moved H3 8.28 mm to (169.7, 114.8)
- moved H1 8.28 mm to (105.2, 114.8)
- moved H4 7.94 mm to (169.7, 45.2)
- moved U1 7.68 mm to (120.8, 91.7)
- moved H2 7.60 mm to (105.4, 45.7)
- moved C2 4.67 mm to (120.7, 63.8)
- moved C1 4.66 mm to (118.1, 96.8)
- renumbered PWR to J1, LORA to U1
Connections:
- J1 pad 1: +5V -> Net-(J1-Pad1)
Routing:
- net +5V: track 50.6 -> 0.00 mm
- net Net-(J2-Pad2): track 18.1 -> 0.00 mm
Other:
- board size 59 x 75 mm -> 75 x 80 mm

Commit message: hopefully done
Parts:
- removed C2: 100n, Capacitor_THT:C_Disc_D3.8mm_W2.6mm_P2.50mm
- added G***: LOGO, EStopFootprints:Paradigm_NameBelow_25.4mm, F.Cu at (122.7, 69.3)
- added LED: LED, LED_THT:LED_D5.0mm, F.Cu at (97.0, 73.4)
- moved Switch1 49.6 mm to (102.9, 89.9)
- moved C1 22.7 mm to (132.6, 114.3)
- moved H4 19.9 mm to (177.5, 63.5)
- moved H2 18.6 mm to (99.8, 63.5)
- moved J2 18.0 mm to (160.6, 67.5)
- moved U1 16.2 mm to (129.8, 105.2)
- moved R1 14.0 mm to (166.1, 76.7)
- moved H3 8.13 mm to (177.8, 114.8)
- moved H1 5.33 mm to (99.8, 114.8)
- moved J1 5.14 mm to (115.3, 102.9)
Connections:
- U1 pad 20: +5V -> unconnected-(U1-Pad20)
- U1 pad 4: GND -> unconnected-(U1-Pad4)
Routing:
- net +5V: track 0.00 -> 139.9 mm
- net Net-(J1-Pad1): track 0.00 -> 22.9 mm
- net Net-(J2-Pad2): track 0.00 -> 16.6 mm
Other:
- board size 75 x 80 mm -> 88.4 x 62 mm

Commit message: Estop review
Parts:
- added R2: 300, Resistor_THT:R_Axial_DIN0207_L6.3mm_D2.5mm_P10.16mm_Horizontal, F.Cu at (113.8, 83.5)
- moved G*** 9.77 mm to (132.4, 69.3)
- moved C1 2.98 mm to (129.8, 113.2)
- moved D1 2.56 mm to (98.2, 71.1), turned to -90 degrees
- moved J1 1.55 mm to (115.3, 104.4)
- renumbered LED to D1
Connections:
- D1 pad 2: +5V -> Net-(D1-Pad2)
- J2 pad 1: +5V -> +3V3
- Switch1 pad 3: GND -> unconnected-(Switch1-Pad3)
- U1 pad 4: unconnected-(U1-Pad4) -> +3V3
Routing:
- net +5V: track 139.9 -> 62.2 mm
- net +3V3: track 0.00 -> 47.3 mm
- net Net-(D1-Pad2): track 0.00 -> 15.7 mm
- net Net-(J1-Pad1): track 22.9 -> 32.5 mm
- net GND: track 0.00 -> 8.08 mm

Commit message: Build Files
Changed lines of the file:
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@@
       (layerselection 0x00010fc_ffffffff)
       (disableapertmacros false)
-      (usegerberextensions false)
-      (usegerberattributes true)
-      (usegerberadvancedattributes true)
-      (creategerberjobfile true)
+      (usegerberextensions true)
+      (usegerberattributes false)
+      (usegerberadvancedattributes false)
+      (creategerberjobfile false)
       (svguseinch false)
       (svgprecision 6)
@@
       (psa4output false)
       (plotreference true)
-      (plotvalue true)
+      (plotvalue false)
       (plotinvisibletext false)
       (sketchpadsonfab false)
-      (subtractmaskfromsilk false)
+      (subtractmaskfromsilk true)
       (outputformat 1)
       (mirror false)
-      (drillshape 1)
+      (drillshape 0)
       (scaleselection 1)
       (outputdirectory "")
@@
     (fp_line (start 0 0) (end 0.75 0.98) (layer "F.Fab") (width 0.1))
     (pad "" np_thru_hole circle (at 1.5 -4.32) (size 3 3) (drill 3) (layers *.Cu *.Mask))
-    (pad "1" thru_hole roundrect (at 0 0) (size 1.5 2.02) (drill 1.02) (layers *.Cu *.Mask) (roundrect_rratio 0.166667)
+    (pad "1" thru_hole roundrect (at 0 0) (size 1.5 2.02) (drill 1.02) (layers *.Cu *.Mask) (roundrect_rratio 0.1666673333)
       (net 39 "+3V3") (pinfunction "Pin_1") (pintype "passive"))
     (pad "2" thru_hole oval (at 3 0) (size 1.5 2.02) (drill 1.02) (layers *.Cu *.Mask)
@@
   (gr_line (start 94.488 120.01) (end 182.88 120) (layer "Edge.Cuts") (width 0.15))
   (gr_line (start 94.488 58) (end 94.488 120.01) (layer "Edge.Cuts") (width 0.15))
-  (gr_text "Paradigm IGVC\nE-Stop TX Rev 1\nNoel Rowsell\n2023\n" (at 155.448 113.538) (layer "F.SilkS")
+  (gr_text "Paradigm IGVC\nE-Stop TX Rev 1\nNoel Rowsell 2023\n" (at 155.448 113.538) (layer "F.SilkS")
     (effects (font (size 1.25 1.25) (thickness 0.15)))
   )
