File: hardware/EStopTX/EStopTX/EStopTX.kicad_sch (KiCad schematic)
At the start: 6 parts, among them J1 USB_B, J2 Conn, U1 Lora_Module

Commit message: Things
Parts:
- C1, C2: footprint Capacitor_THT:CP_Radial_D4.0mm_P2.00mm -> Capacitor_THT:C_Disc_D3.8mm_W2.6mm_P2.50mm; Digikey (none) -> BC1084CT-ND
- U1: footprint controlLib:Lora_Module -> EStopFootprints:Lora_Module
Connections:
- net +5V: now also C1.2; no longer C1.1
- net GND: now also C1.1; no longer C1.2
Changed lines of the file:
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@@
     (property "Reference" "U1" (id 0) (at 177.8 34.29 0))
     (property "Value" "Lora_Module" (id 1) (at 177.8 36.83 0))
-    (property "Footprint" "controlLib:Lora_Module" (id 2) (at 177.8 24.13 0)
+    (property "Footprint" "EStopFootprints:Lora_Module" (id 2) (at 177.8 24.13 0)
       (effects (font (size 1.27 1.27)) hide)
     )
@@
     (pin "1")
   )
+  (symbol (lib_id "Device:C") (at 196.85 52.07 0) (unit 1)
+    (in_bom yes) (on_board yes) (fields_autoplaced)
+    (property "Reference" "C2" (id 0) (at 200.66 50.7999 0)
+      (effects (font (size 1.27 1.27)) (justify left))
+    )
+    (property "Value" "100n" (id 1) (at 200.66 53.3399 0)
+      (effects (font (size 1.27 1.27)) (justify left))
+    )
+    (property "Footprint" "Capacitor_THT:C_Disc_D3.8mm_W2.6mm_P2.50mm" (id 2) (at 197.8152 55.88 0)
+      (effects (font (size 1.27 1.27)) hide)
+    )
+    (property "Datasheet" "https://www.vishay.com/docs/45171/kseries.pdf" (id 3) (at 196.85 52.07 0)
+      (effects (font (size 1.27 1.27)) hide)
+    )
+    (property "Digikey" "BC1084CT-ND" (id 4) (at 196.85 52.07 0)
+      (effects (font (size 1.27 1.27)) hide)
+    )
+    (pin "1")
+    (pin "2")
+  )
   (symbol (lib_id "power:GND") (at 162.56 52.07 0) (unit 1)
     (in_bom yes) (on_board yes) (fields_autoplaced)
@@
     (pin "1")
   )
-  (symbol (lib_id "Device:C") (at 152.4 52.07 0) (unit 1)
-    (in_bom yes) (on_board yes) (fields_autoplaced)
-    (property "Reference" "C1" (id 0) (at 156.21 50.7999 0)
-      (effects (font (size 1.27 1.27)) (justify left))
-    )
-    (property "Value" "100n" (id 1) (at 156.21 53.3399 0)
-      (effects (font (size 1.27 1.27)) (justify left))
-    )
-    (property "Footprint" "Capacitor_THT:CP_Radial_D4.0mm_P2.00mm" (id 2) (at 153.3652 55.88 0)
-      (effects (font (size 1.27 1.27)) hide)
-    )
-    (property "Datasheet" "~" (id 3) (at 152.4 52.07 0)
-      (effects (font (size 1.27 1.27)) hide)
-    )
-    (pin "1")
-    (pin "2")
-  )
-  (symbol (lib_id "Device:C") (at 196.85 52.07 0) (unit 1)
-    (in_bom yes) (on_board yes) (fields_autoplaced)
-    (property "Reference" "C2" (id 0) (at 200.66 50.7999 0)
-      (effects (font (size 1.27 1.27)) (justify left))
-    )
-    (property "Value" "100n" (id 1) (at 200.66 53.3399 0)
-      (effects (font (size 1.27 1.27)) (justify left))
-    )
-    (property "Footprint" "Capacitor_THT:CP_Radial_D4.0mm_P2.00mm" (id 2) (at 197.8152 55.88 0)
-      (effects (font (size 1.27 1.27)) hide)
-    )
-    (property "Datasheet" "~" (id 3) (at 196.85 52.07 0)
+  (symbol (lib_id "Device:C") (at 152.4 52.07 0) (mirror x) (unit 1)
+    (in_bom yes) (on_board yes) (fields_autoplaced)
+    (property "Reference" "C1" (id 0) (at 148.59 50.7999 0)
+      (effects (font (size 1.27 1.27)) (justify right))
+    )
+    (property "Value" "100n" (id 1) (at 148.59 53.3399 0)
+      (effects (font (size 1.27 1.27)) (justify right))
+    )
+    (property "Footprint" "Capacitor_THT:C_Disc_D3.8mm_W2.6mm_P2.50mm" (id 2) (at 153.3652 48.26 0)
+      (effects (font (size 1.27 1.27)) hide)
+    )
+    (property "Datasheet" "https://www.vishay.com/docs/45171/kseries.pdf" (id 3) (at 152.4 52.07 0)
+      (effects (font (size 1.27 1.27)) hide)
+    )
+    (property "Digikey" "BC1084CT-ND" (id 4) (at 152.4 52.07 0)
       (effects (font (size 1.27 1.27)) hide)
     )
@@
     )
     (path "/8b7d6f14-c49a-4850-af30-959f0653bde1"
-      (reference "C1") (unit 1) (value "100n") (footprint "Capacitor_THT:CP_Radial_D4.0mm_P2.00mm")
-    )
-    (path "/d119cdca-3658-4764-b770-afd1bc022af4"
-      (reference "C2") (unit 1) (value "100n") (footprint "Capacitor_THT:CP_Radial_D4.0mm_P2.00mm")
+      (reference "C1") (unit 1) (value "100n") (footprint "Capacitor_THT:C_Disc_D3.8mm_W2.6mm_P2.50mm")
+    )
+    (path "/64ebb9af-411b-4c4f-bc60-2133502e0dad"
+      (reference "C2") (unit 1) (value "100n") (footprint "Capacitor_THT:C_Disc_D3.8mm_W2.6mm_P2.50mm")
     )
     (path "/391374e5-5ab6-469b-a57a-4857fd6856b0"
@@
     )
     (path "/3dced294-be75-40b1-9d68-62c572fa8849"
-      (reference "U1") (unit 1) (value "Lora_Module") (footprint "controlLib:Lora_Module")
-    )
-  )
+      (reference "U1") (unit 1) (value "Lora_Module") (footprint "EStopFootprints:Lora_Module")
+    )
+  )

Commit message: maybe done?
Parts:
- added H1, H2, H3, H4: MountingHole, MountingHole:MountingHole_3.2mm_M3_Pad_Via, symbol Mechanical:MountingHole
Changed lines of the file:
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@@
     (stroke (width 0) (type default) (color 0 0 0 0))
+  )
+  (symbol (lib_id "Mechanical:MountingHole") (at 90.17 35.56 0) (unit 1)
+    (in_bom yes) (on_board yes) (fields_autoplaced)
+    (property "Reference" "H1" (id 0) (at 92.71 34.2899 0)
+      (effects (font (size 1.27 1.27)) (justify left))
+    )
+    (property "Value" "MountingHole" (id 1) (at 92.71 36.8299 0)
+      (effects (font (size 1.27 1.27)) (justify left))
+    )
+    (property "Footprint" "MountingHole:MountingHole_3.2mm_M3_Pad_Via" (id 2) (at 90.17 35.56 0)
+      (effects (font (size 1.27 1.27)) hide)
+    )
+    (property "Datasheet" "~" (id 3) (at 90.17 35.56 0)
+      (effects (font (size 1.27 1.27)) hide)
+    )
   )
   (symbol (lib_id "power:+5V") (at 152.4 45.72 0) (unit 1)
@@
     )
     (pin "1")
+  )
+  (symbol (lib_id "Mechanical:MountingHole") (at 90.17 50.8 0) (unit 1)
+    (in_bom yes) (on_board yes) (fields_autoplaced)
+    (property "Reference" "H4" (id 0) (at 92.71 49.5299 0)
+      (effects (font (size 1.27 1.27)) (justify left))
+    )
+    (property "Value" "MountingHole" (id 1) (at 92.71 52.0699 0)
+      (effects (font (size 1.27 1.27)) (justify left))
+    )
+    (property "Footprint" "MountingHole:MountingHole_3.2mm_M3_Pad_Via" (id 2) (at 90.17 50.8 0)
+      (effects (font (size 1.27 1.27)) hide)
+    )
+    (property "Datasheet" "~" (id 3) (at 90.17 50.8 0)
+      (effects (font (size 1.27 1.27)) hide)
+    )
   )
   (symbol (lib_id "power:GND") (at 152.4 57.15 0) (unit 1)
@@
     (pin "2")
   )
+  (symbol (lib_id "Mechanical:MountingHole") (at 90.17 45.72 0) (unit 1)
+    (in_bom yes) (on_board yes) (fields_autoplaced)
+    (property "Reference" "H3" (id 0) (at 92.71 44.4499 0)
+      (effects (font (size 1.27 1.27)) (justify left))
+    )
+    (property "Value" "MountingHole" (id 1) (at 92.71 46.9899 0)
+      (effects (font (size 1.27 1.27)) (justify left))
+    )
+    (property "Footprint" "MountingHole:MountingHole_3.2mm_M3_Pad_Via" (id 2) (at 90.17 45.72 0)
+      (effects (font (size 1.27 1.27)) hide)
+    )
+    (property "Datasheet" "~" (id 3) (at 90.17 45.72 0)
+      (effects (font (size 1.27 1.27)) hide)
+    )
+  )
+  (symbol (lib_id "Mechanical:MountingHole") (at 90.17 40.64 0) (unit 1)
+    (in_bom yes) (on_board yes) (fields_autoplaced)
+    (property "Reference" "H2" (id 0) (at 92.71 39.3699 0)
+      (effects (font (size 1.27 1.27)) (justify left))
+    )
+    (property "Value" "MountingHole" (id 1) (at 92.71 41.9099 0)
+      (effects (font (size 1.27 1.27)) (justify left))
+    )
+    (property "Footprint" "MountingHole:MountingHole_3.2mm_M3_Pad_Via" (id 2) (at 90.17 40.64 0)
+      (effects (font (size 1.27 1.27)) hide)
+    )
+    (property "Datasheet" "~" (id 3) (at 90.17 40.64 0)
+      (effects (font (size 1.27 1.27)) hide)
+    )
+  )
   (symbol (lib_id "power:+5V") (at 205.74 78.74 0) (unit 1)
     (in_bom yes) (on_board yes) (fields_autoplaced)
@@
       (reference "C2") (unit 1) (value "100n") (footprint "Capacitor_THT:C_Disc_D3.8mm_W2.6mm_P2.50mm")
     )
+    (path "/0283c443-8942-4f6a-98b3-668972153b58"
+      (reference "H1") (unit 1) (value "MountingHole") (footprint "MountingHole:MountingHole_3.2mm_M3_Pad_Via")
+    )
+    (path "/b9c07d33-22f5-479c-98a4-5f430ef98dcd"
+      (reference "H2") (unit 1) (value "MountingHole") (footprint "MountingHole:MountingHole_3.2mm_M3_Pad_Via")
+    )
+    (path "/90c0c2bc-2fe6-4be0-9959-cc7afd1d1c6c"
+      (reference "H3") (unit 1) (value "MountingHole") (footprint "MountingHole:MountingHole_3.2mm_M3_Pad_Via")
+    )
+    (path "/14089165-9181-47c7-9056-2c3dc1216a42"
+      (reference "H4") (unit 1) (value "MountingHole") (footprint "MountingHole:MountingHole_3.2mm_M3_Pad_Via")
+    )
     (path "/391374e5-5ab6-469b-a57a-4857fd6856b0"

Commit message: changes
Parts:
- added Switch1: L102021ML04Q, EStopFootprints:SW_L102021ML04Q, symbol EStopTX_Lib:L102021ML04Q
Connections:
- net +5V: now also Switch1.2; no longer J1.1 (VBUS)
- net GND: now also Switch1.3
- new net: J1.1 (VBUS), Switch1.1
Changed lines of the file:
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@@
+    (stroke (width 0) (type default) (color 0 0 0 0))
+  )
+  (wire (pts (xy 121.92 43.18) (xy 121.92 31.75))
     (stroke (width 0) (type default) (color 0 0 0 0))
   )
@@
     (stroke (width 0) (type default) (color 0 0 0 0))
   )
+  (wire (pts (xy 127 36.83) (xy 130.81 36.83))
+    (stroke (width 0) (type default) (color 0 0 0 0))
+  )
   (wire (pts (xy 196.85 57.15) (xy 196.85 55.88))
     (stroke (width 0) (type default) (color 0 0 0 0))
@@
     (stroke (width 0) (type default) (color 0 0 0 0))
   )
-  (wire (pts (xy 121.92 43.18) (xy 125.73 43.18))
+  (wire (pts (xy 121.92 31.75) (xy 130.81 31.75))
+    (stroke (width 0) (type default) (color 0 0 0 0))
+  )
+  (wire (pts (xy 127 34.29) (xy 130.81 34.29))
     (stroke (width 0) (type default) (color 0 0 0 0))
   )
@@
     (stroke (width 0) (type default) (color 0 0 0 0))
   )
-  (wire (pts (xy 125.73 43.18) (xy 125.73 40.64))
-    (stroke (width 0) (type default) (color 0 0 0 0))
-  )
   (wire (pts (xy 152.4 45.72) (xy 166.37 45.72))
     (stroke (width 0) (type default) (color 0 0 0 0))
@@
   )
   (symbol (lib_id "power:+5V") (at 152.4 45.72 0) (unit 1)
-    (in_bom yes) (on_board yes) (fields_autoplaced)
+    (in_bom yes) (on_board yes)
     (property "Reference" "#PWR0102" (id 0) (at 152.4 49.53 0)
       (effects (font (size 1.27 1.27)) hide)
@@
     (pin "1")
   )
+  (symbol (lib_id "power:+5V") (at 127 34.29 0) (unit 1)
+    (in_bom yes) (on_board yes)
+    (property "Reference" "#PWR0103" (id 0) (at 127 38.1 0)
+      (effects (font (size 1.27 1.27)) hide)
+    )
+    (property "Value" "+5V" (id 1) (at 127 29.21 0))
+    (property "Footprint" "" (id 2) (at 127 34.29 0)
+      (effects (font (size 1.27 1.27)) hide)
+    )
+    (property "Datasheet" "" (id 3) (at 127 34.29 0)
+      (effects (font (size 1.27 1.27)) hide)
+    )
+    (pin "1")
+  )
   (symbol (lib_id "power:+5V") (at 196.85 45.72 0) (unit 1)
     (in_bom yes) (on_board yes) (fields_autoplaced)
@@
     (pin "1")
   )
+  (symbol (lib_id "EStopTX_Lib:L102021ML04Q") (at 140.97 34.29 0) (unit 1)
+    (in_bom yes) (on_board yes) (fields_autoplaced)
+    (property "Reference" "Switch1" (id 0) (at 147.32 33.0199 0)
+      (effects (font (size 1.27 1.27)) (justify left))
+    )
+    (property "Value" "L102021ML04Q" (id 1) (at 147.32 35.5599 0)
+      (effects (font (size 1.27 1.27)) (justify left))
+    )
+    (property "Footprint" "EStopFootprints:SW_L102021ML04Q" (id 2) (at 140.97 34.29 0)
+      (effects (font (size 1.27 1.27)) (justify left bottom) hide)
+    )
+    (property "Datasheet" "" (id 3) (at 140.97 34.29 0)
+      (effects (font (size 1.27 1.27)) (justify left bottom) hide)
+    )
+    (property "Availability" "In Stock" (id 4) (at 140.97 34.29 0)
+      (effects (font (size 1.27 1.27)) (justify left bottom) hide)
+    )
+    (property "Price" "None" (id 5) (at 140.97 34.29 0)
+      (effects (font (size 1.27 1.27)) (justify left bottom) hide)
+    )
+    (property "MF" "C&K" (id 6) (at 140.97 34.29 0)
+      (effects (font (size 1.27 1.27)) (justify left bottom) hide)
+    )
+    (property "Description" "\\nSlide Switch SPDT Through Hole, Right Angle\\n" (id 7) (at 140.97 34.29 0)
+      (effects (font (size 1.27 1.27)) (justify left bottom) hide)
+    )
+    (property "Package" "None" (id 8) (at 140.97 34.29 0)
+      (effects (font (size 1.27 1.27)) (justify left bottom) hide)
+    )
+    (property "MP" "L102021ML04Q" (id 9) (at 140.97 34.29 0)
+      (effects (font (size 1.27 1.27)) (justify left bottom) hide)
+    )
+    (pin "1")
+    (pin "2")
+    (pin "3")
+  )
   (symbol (lib_id "Mechanical:MountingHole") (at 90.17 50.8 0) (unit 1)
     (in_bom yes) (on_board yes) (fields_autoplaced)
@@
     (pin "1")
   )
-  (symbol (lib_id "power:+5V") (at 125.73 40.64 0) (unit 1)
-    (in_bom yes) (on_board yes) (fields_autoplaced)
-    (property "Reference" "#PWR0103" (id 0) (at 125.73 44.45 0)
-      (effects (font (size 1.27 1.27)) hide)
-    )
-    (property "Value" "+5V" (id 1) (at 125.73 35.56 0))
-    (property "Footprint" "" (id 2) (at 125.73 40.64 0)
-      (effects (font (size 1.27 1.27)) hide)
-    )
-    (property "Datasheet" "" (id 3) (at 125.73 40.64 0)
+  (symbol (lib_id "power:GND") (at 127 36.83 0) (unit 1)
+    (in_bom yes) (on_board yes) (fields_autoplaced)
+    (property "Reference" "#PWR0113" (id 0) (at 127 43.18 0)
+      (effects (font (size 1.27 1.27)) hide)
+    )
+    (property "Value" "GND" (id 1) (at 127 41.91 0))
+    (property "Footprint" "" (id 2) (at 127 36.83 0)
+      (effects (font (size 1.27 1.27)) hide)
+    )
+    (property "Datasheet" "" (id 3) (at 127 36.83 0)
       (effects (font (size 1.27 1.27)) hide)
     )
@@
       (reference "#PWR0102") (unit 1) (value "+5V") (footprint "")
     )
-    (path "/36c71436-dcee-428f-99af-5b106fa75479"
+    (path "/0730e5ff-2f90-4317-bcc2-b7e95a27c697"
       (reference "#PWR0103") (unit 1) (value "+5V") (footprint "")
     )
@@
       (reference "#PWR0112") (unit 1) (value "GND") (footprint "")
     )
+    (path "/15b40cbe-e4af-4aff-aba4-b6b58c26046f"
+      (reference "#PWR0113") (unit 1) (value "GND") (footprint "")
+    )
     (path "/8b7d6f14-c49a-4850-af30-959f0653bde1"
       (reference "C1") (unit 1) (value "100n") (footprint "Capacitor_THT:C_Disc_D3.8mm_W2.6mm_P2.50mm")
@@
       (reference "R1") (unit 1) (value "4.7k") (footprint "Resistor_THT:R_Axial_DIN0207_L6.3mm_D2.5mm_P10.16mm_Horizontal")
     )
+    (path "/0fc76667-385a-49c2-a597-5c0a808fefb8"
+      (reference "Switch1") (unit 1) (value "L102021ML04Q") (footprint "EStopFootprints:SW_L102021ML04Q")
+    )
     (path "/3dced294-be75-40b1-9d68-62c572fa8849"

Commit message: hopefully done
Parts:
- removed C2: 100n, Capacitor_THT:C_Disc_D3.8mm_W2.6mm_P2.50mm, symbol Device:C
- added D1: LED, LED_THT:LED_D5.0mm, symbol Device:LED
Connections:
- net +5V: now also D1.2 (A); no longer U1.20 (5V)
- net GND: now also D1.1 (K); no longer U1.4 (GND)
- no-connect marks 32 -> 34
