File: hardware/EStopTX/EStopTX/EStopTX.kicad_sch (KiCad schematic)
At the start: 11 parts, among them J1 USB_B, J2 Conn, U1 Lora_Module

Commit message: Estop review
Parts:
- added R2: 300, Resistor_THT:R_Axial_DIN0207_L6.3mm_D2.5mm_P10.16mm_Horizontal, symbol Device:R
- Switch1: Digikey (none) -> CKC5102-ND
Connections:
- net +5V: now also R2.1; no longer D1.2 (A), J2.1 (Pin_1)
- net GND: no longer Switch1.3
- net +3V3: now reaches U1.4 (VEXT)
- net +3V3: now also J2.1 (Pin_1)
- new net: D1.2 (A), R2.2
- no-connect marks 34 -> 33
Changed lines of the file:
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@@
   (junction (at 152.4 45.72) (diameter 0) (color 0 0 0 0)
   )
-  (junction (at 125.73 57.15) (diameter 0) (color 0 0 0 0)
+  (junction (at 125.73 45.72) (diameter 0) (color 0 0 0 0)
   )
   (no_connect (at 189.23 83.82))
@@
   (no_connect (at 189.23 68.58))
   (no_connect (at 189.23 60.96))
-  (no_connect (at 166.37 50.8))
   (no_connect (at 166.37 53.34))
   (no_connect (at 189.23 45.72))
@@
     (stroke (width 0) (type default) (color 0 0 0 0))
   )
+  (wire (pts (xy 125.73 49.53) (xy 125.73 45.72))
+    (stroke (width 0) (type default) (color 0 0 0 0))
+  )
   (wire (pts (xy 121.92 43.18) (xy 121.92 31.75))
     (stroke (width 0) (type default) (color 0 0 0 0))
@@
     (stroke (width 0) (type default) (color 0 0 0 0))
   )
-  (wire (pts (xy 129.54 36.83) (xy 130.81 36.83))
+  (wire (pts (xy 162.56 50.8) (xy 166.37 50.8))
     (stroke (width 0) (type default) (color 0 0 0 0))
   )
@@
     (stroke (width 0) (type default) (color 0 0 0 0))
   )
+  (wire (pts (xy 203.2 78.74) (xy 203.2 77.47))
+    (stroke (width 0) (type default) (color 0 0 0 0))
+  )
+  (wire (pts (xy 125.73 45.72) (xy 129.54 45.72))
+    (stroke (width 0) (type default) (color 0 0 0 0))
+  )
+  (wire (pts (xy 129.54 44.45) (xy 129.54 45.72))
+    (stroke (width 0) (type default) (color 0 0 0 0))
+  )
   (wire (pts (xy 163.83 36.83) (xy 166.37 36.83))
     (stroke (width 0) (type default) (color 0 0 0 0))
@@
     (stroke (width 0) (type default) (color 0 0 0 0))
   )
+  (wire (pts (xy 203.2 78.74) (xy 205.74 78.74))
+    (stroke (width 0) (type default) (color 0 0 0 0))
+  )
   (wire (pts (xy 121.92 31.75) (xy 130.81 31.75))
     (stroke (width 0) (type default) (color 0 0 0 0))
   )
-  (wire (pts (xy 125.73 34.29) (xy 125.73 57.15))
+  (wire (pts (xy 125.73 34.29) (xy 125.73 45.72))
     (stroke (width 0) (type default) (color 0 0 0 0))
   )
@@
   )
   (wire (pts (xy 152.4 45.72) (xy 166.37 45.72))
-    (stroke (width 0) (type default) (color 0 0 0 0))
-  )
-  (wire (pts (xy 129.54 57.15) (xy 129.54 55.88))
-    (stroke (width 0) (type default) (color 0 0 0 0))
-  )
-  (wire (pts (xy 125.73 57.15) (xy 129.54 57.15))
     (stroke (width 0) (type default) (color 0 0 0 0))
   )
@@
     (pin "1")
   )
+  (symbol (lib_id "power:+3V3") (at 162.56 50.8 0) (unit 1)
+    (in_bom yes) (on_board yes)
+    (property "Reference" "#PWR0106" (id 0) (at 162.56 54.61 0)
+      (effects (font (size 1.27 1.27)) hide)
+    )
+    (property "Value" "+3V3" (id 1) (at 162.56 46.99 0))
+    (property "Footprint" "" (id 2) (at 162.56 50.8 0)
+      (effects (font (size 1.27 1.27)) hide)
+    )
+    (property "Datasheet" "" (id 3) (at 162.56 50.8 0)
+      (effects (font (size 1.27 1.27)) hide)
+    )
+    (pin "1")
+  )
   (symbol (lib_id "EStopTX_Lib:L102021ML04Q") (at 140.97 34.29 0) (unit 1)
     (in_bom yes) (on_board yes) (fields_autoplaced)
@@
       (effects (font (size 1.27 1.27)) (justify left bottom) hide)
     )
-    (property "Datasheet" "" (id 3) (at 140.97 34.29 0)
+    (property "Datasheet" "https://www.ckswitches.com/media/1423/l.pdf" (id 3) (at 140.97 34.29 0)
       (effects (font (size 1.27 1.27)) (justify left bottom) hide)
     )
@@
     (property "MP" "L102021ML04Q" (id 9) (at 140.97 34.29 0)
       (effects (font (size 1.27 1.27)) (justify left bottom) hide)
+    )
+    (property "Digikey" "CKC5102-ND" (id 10) (at 140.97 34.29 0)
+      (effects (font (size 1.27 1.27)) hide)
     )
     (pin "1")
@@
     (pin "1")
   )
-  (symbol (lib_id "power:GND") (at 129.54 36.83 0) (unit 1)
-    (in_bom yes) (on_board yes)
-    (property "Reference" "#PWR0113" (id 0) (at 129.54 43.18 0)
-      (effects (font (size 1.27 1.27)) hide)
-    )
-    (property "Value" "GND" (id 1) (at 129.54 40.64 0))
-    (property "Footprint" "" (id 2) (at 129.54 36.83 0)
-      (effects (font (size 1.27 1.27)) hide)
-    )
-    (property "Datasheet" "" (id 3) (at 129.54 36.83 0)
-      (effects (font (size 1.27 1.27)) hide)
-    )
-    (pin "1")
+  (symbol (lib_id "Device:R") (at 125.73 53.34 0) (unit 1)
+    (in_bom yes) (on_board yes) (fields_autoplaced)
+    (property "Reference" "R2" (id 0) (at 128.27 52.0699 0)
+      (effects (font (size 1.27 1.27)) (justify left))
+    )
+    (property "Value" "300" (id 1) (at 128.27 54.6099 0)
+      (effects (font (size 1.27 1.27)) (justify left))
+    )
+    (property "Footprint" "Resistor_THT:R_Axial_DIN0207_L6.3mm_D2.5mm_P10.16mm_Horizontal" (id 2) (at 123.952 53.34 90)
+      (effects (font (size 1.27 1.27)) hide)
+    )
+    (property "Datasheet" "~" (id 3) (at 125.73 53.34 0)
+      (effects (font (size 1.27 1.27)) hide)
+    )
+    (pin "1")
+    (pin "2")
   )
   (symbol (lib_id "power:GND") (at 114.3 63.5 0) (unit 1)
@@
   (symbol (lib_id "power:GND") (at 125.73 68.58 0) (unit 1)
     (in_bom yes) (on_board yes) (fields_autoplaced)
-    (property "Reference" "#PWR?" (id 0) (at 125.73 74.93 0)
+    (property "Reference" "#PWR0107" (id 0) (at 125.73 74.93 0)
       (effects (font (size 1.27 1.27)) hide)
     )
@@
     (pin "2")
   )
-  (symbol (lib_id "power:+5V") (at 129.54 55.88 0) (unit 1)
-    (in_bom yes) (on_board yes) (fields_autoplaced)
-    (property "Reference" "#PWR?" (id 0) (at 129.54 59.69 0)
-      (effects (font (size 1.27 1.27)) hide)
-    )
-    (property "Value" "+5V" (id 1) (at 129.54 50.8 0))
-    (property "Footprint" "" (id 2) (at 129.54 55.88 0)
-      (effects (font (size 1.27 1.27)) hide)
-    )
-    (property "Datasheet" "" (id 3) (at 129.54 55.88 0)
+  (symbol (lib_id "power:+5V") (at 129.54 44.45 0) (unit 1)
+    (in_bom yes) (on_board yes)
+    (property "Reference" "#PWR0109" (id 0) (at 129.54 48.26 0)
+      (effects (font (size 1.27 1.27)) hide)
+    )
+    (property "Value" "+5V" (id 1) (at 129.54 40.64 0))
+    (property "Footprint" "" (id 2) (at 129.54 44.45 0)
+      (effects (font (size 1.27 1.27)) hide)
+    )
+    (property "Datasheet" "" (id 3) (at 129.54 44.45 0)
       (effects (font (size 1.27 1.27)) hide)
     )
@@
     )
   )
-  (symbol (lib_id "power:+5V") (at 205.74 78.74 0) (unit 1)
-    (in_bom yes) (on_board yes) (fields_autoplaced)
-    (property "Reference" "#PWR0111" (id 0) (at 205.74 82.55 0)
-      (effects (font (size 1.27 1.27)) hide)
-    )
-    (property "Value" "+5V" (id 1) (at 205.74 73.66 0))
-    (property "Footprint" "" (id 2) (at 205.74 78.74 0)
-      (effects (font (size 1.27 1.27)) hide)
-    )
-    (property "Datasheet" "" (id 3) (at 205.74 78.74 0)
+  (symbol (lib_id "power:+3V3") (at 203.2 77.47 0) (unit 1)
+    (in_bom yes) (on_board yes) (fields_autoplaced)
+    (property "Reference" "#PWR0103" (id 0) (at 203.2 81.28 0)
+      (effects (font (size 1.27 1.27)) hide)
+    )
+    (property "Value" "+3V3" (id 1) (at 203.2 72.39 0))
+    (property "Footprint" "" (id 2) (at 203.2 77.47 0)
+      (effects (font (size 1.27 1.27)) hide)
+    )
+    (property "Datasheet" "" (id 3) (at 203.2 77.47 0)
       (effects (font (size 1.27 1.27)) hide)
     )
@@
       (reference "#PWR0102") (unit 1) (value "+5V") (footprint "")
     )
+    (path "/f0dfac2f-eb95-4536-8e82-94453fe2e407"
+      (reference "#PWR0103") (unit 1) (value "+3V3") (footprint "")
+    )
     (path "/37d87525-beac-47cd-82a9-77bd23406538"
       (reference "#PWR0104") (unit 1) (value "GND") (footprint "")
@@
       (reference "#PWR0105") (unit 1) (value "GND") (footprint "")
     )
+    (path "/05f143e8-e353-438e-8ee8-d27db0558010"
+      (reference "#PWR0106") (unit 1) (value "+3V3") (footprint "")
+    )
+    (path "/732bee8f-0697-4c19-b09b-57850535cddd"
+      (reference "#PWR0107") (unit 1) (value "GND") (footprint "")
+    )
     (path "/8100dc2f-4887-4285-95cb-4a34a84c9d06"
       (reference "#PWR0108") (unit 1) (value "GND") (footprint "")
     )
+    (path "/a9a103a2-341d-4f69-a250-367e34caee5b"
+      (reference "#PWR0109") (unit 1) (value "+5V") (footprint "")
+    )
     (path "/79876e3a-4369-446c-942c-204a0b5e0db3"
       (reference "#PWR0110") (unit 1) (value "GND") (footprint "")
     )
-    (path "/d7b805cf-fefe-44db-bc4a-3c4447e7f429"
-      (reference "#PWR0111") (unit 1) (value "+5V") (footprint "")
-    )
     (path "/15b036d1-64d5-49f4-a7fe-71d07bb90780"
       (reference "#PWR0112") (unit 1) (value "GND") (footprint "")
     )
-    (path "/15b40cbe-e4af-4aff-aba4-b6b58c26046f"
-      (reference "#PWR0113") (unit 1) (value "GND") (footprint "")
-    )
-    (path "/732bee8f-0697-4c19-b09b-57850535cddd"
-      (reference "#PWR?") (unit 1) (value "GND") (footprint "")
-    )
-    (path "/a9a103a2-341d-4f69-a250-367e34caee5b"
-      (reference "#PWR?") (unit 1) (value "+5V") (footprint "")
-    )
     (path "/8b7d6f14-c49a-4850-af30-959f0653bde1"
       (reference "C1") (unit 1) (value "100n") (footprint "Capacitor_THT:C_Disc_D3.8mm_W2.6mm_P2.50mm")
@@
       (reference "R1") (unit 1) (value "4.7k") (footprint "Resistor_THT:R_Axial_DIN0207_L6.3mm_D2.5mm_P10.16mm_Horizontal")
     )
+    (path "/28ae482b-4217-4a87-ab08-7a3b95442bec"
+      (reference "R2") (unit 1) (value "300") (footprint "Resistor_THT:R_Axial_DIN0207_L6.3mm_D2.5mm_P10.16mm_Horizontal")
+    )
     (path "/0fc76667-385a-49c2-a597-5c0a808fefb8"
