File: hardware/PowerDistributionBoard/PowerDistributionBoard/PowerDistributionBoard.kicad_pcb (KiCad board)
At the start: 4 copper layers, 180 x 120 mm, 129 parts, among them J1 Battery, J10 MOTOR2_PWR, J11 Router, J2 FAN 1, J3 FAN 2, J4 FAN 3, J5 FAN 4, J6 Inverter, J7 Control Board, J8 Conn_01x02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

Commit message: Finish adding assembly PNs
Parts:
- added FID1: Fiducial, Fiducial:Fiducial_1mm_Mask2mm, F.Cu at (56.2, 28.9)
- added FID2: Fiducial, Fiducial:Fiducial_1mm_Mask2mm, F.Cu at (183.8, 28.9)
- added FID3: Fiducial, Fiducial:Fiducial_1mm_Mask2mm, F.Cu at (56.6, 141.2)
- added FID4: Fiducial, Fiducial:Fiducial_1mm_Mask2mm, F.Cu at (203.6, 141.2)
- R15, R16: value DNP -> ?
Other:
- board text added: "CTRL BOARD PWR"
- board text added: "MOTOR 1 PWR"
- board text added: "MOTOR 2 PWR"
- board text added: "ROUTER"

Commit message: Build Files
Other:
- board text added: "JLCJLCJLCJLC"
